File: schematics/board/SP1.sch (EAGLE design)
At the start: 12 parts

Commit message: развёл плату солнечных панелей(на деньги)
Parts:
- U$1, U$2: value SOLAR-2_0 -> SOLAR-2_1; device CanCubeSat:SOLAR-2_0 -> CanCubeSat:SOLAR-2_1
Changed lines of the file:
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@@
 <?xml version="1.0" encoding="utf-8"?>
 <!DOCTYPE eagle SYSTEM "eagle.dtd">
-<eagle version="9.4.2">
+<eagle version="9.6.2">
 <drawing>
 <settings>
-<setting alwaysvectorfont="yes"/>
+<setting alwaysvectorfont="no"/>
 <setting verticaltext="up"/>
 </settings>
@@
 </classes>
 <parts>
-<part name="U$1" library="CanCubeSat" deviceset="SOLAR-2" device="_0"/>
-<part name="U$2" library="CanCubeSat" deviceset="SOLAR-2" device="_0"/>
+<part name="U$1" library="CanCubeSat" deviceset="SOLAR-2" device="_1" value="SOLAR-2_1"/>
+<part name="U$2" library="CanCubeSat" deviceset="SOLAR-2" device="_1" value="SOLAR-2_1"/>
 <part name="U$3" library="CanCubeSat" deviceset="SOLAR-2" device="_0"/>
 <part name="U$4" library="CanCubeSat" deviceset="SOLAR-2" device="_0"/>
