File: schematics/board/SP2.sch (EAGLE design)
At the start: 12 parts

Commit message: развёл плату солнечных панелей(на деньги)
Parts:
- added JP2: (no value), pinhead:PINHD-1X2
- U$1, U$2: value SOLAR-2_0 -> SOLAR-2_1; device CanCubeSat:SOLAR-2_0 -> CanCubeSat:SOLAR-2_1
Connections:
- new net SP+-: C1.2, D4.C, JP2.1, LED1.C, U$4.OUT
- net SP-: now also JP2.2; no longer C1.2, D4.C, LED1.C, U$4.OUT
Other:
- moved on the sheet: JP1
Changed lines of the file:
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@@
 <?xml version="1.0" encoding="utf-8"?>
 <!DOCTYPE eagle SYSTEM "eagle.dtd">
-<eagle version="9.4.2">
+<eagle version="9.6.2">
 <drawing>
 <settings>
-<setting alwaysvectorfont="yes"/>
+<setting alwaysvectorfont="no"/>
 <setting verticaltext="up"/>
 </settings>
@@
 </classes>
 <parts>
-<part name="U$1" library="CanCubeSat" deviceset="SOLAR-2" device="_0"/>
-<part name="U$2" library="CanCubeSat" deviceset="SOLAR-2" device="_0"/>
+<part name="U$1" library="CanCubeSat" deviceset="SOLAR-2" device="_1" value="SOLAR-2_1"/>
+<part name="U$2" library="CanCubeSat" deviceset="SOLAR-2" device="_1" value="SOLAR-2_1"/>
 <part name="U$3" library="CanCubeSat" deviceset="SOLAR-2" device="_0"/>
 <part name="U$4" library="CanCubeSat" deviceset="SOLAR-2" device="_0"/>
@@
 <part name="D4" library="diode" library_urn="urn:adsk.eagle:library:210" deviceset="MBR0520LT" device="" package3d_urn="urn:adsk.eagle:package:43420/1"/>
 <part name="LED1" library="led" library_urn="urn:adsk.eagle:library:259" deviceset="LED" device="CHIP-LED0603" package3d_urn="urn:adsk.eagle:package:15819/3"/>
+<part name="JP2" library="pinhead" library_urn="urn:adsk.eagle:library:325" deviceset="PINHD-1X2" device="" package3d_urn="urn:adsk.eagle:package:22435/2"/>
 </parts>
 <sheets>
@@
 <attribute name="VALUE" x="20.32" y="23.0886" size="1.778" layer="96"/>
 </instance>
-<instance part="JP1" gate="G$1" x="35.56" y="-27.94" smashed="yes" rot="R270">
-<attribute name="NAME" x="41.275" y="-21.59" size="1.778" layer="95" rot="R270"/>
-<attribute name="VALUE" x="30.48" y="-21.59" size="1.778" layer="96" rot="R270"/>
+<instance part="JP1" gate="G$1" x="25.4" y="-27.94" smashed="yes" rot="R270">
+<attribute name="NAME" x="31.115" y="-21.59" size="1.778" layer="95" rot="R270"/>
+<attribute name="VALUE" x="20.32" y="-21.59" size="1.778" layer="96" rot="R270"/>
 </instance>
 <instance part="D2" gate="G$1" x="30.48" y="25.4" smashed="yes">
@@
 <attribute name="NAME" x="50.292" y="13.716" size="1.778" layer="95" rot="R180"/>
 <attribute name="VALUE" x="50.292" y="15.875" size="1.778" layer="96" rot="R180"/>
+</instance>
+<instance part="JP2" gate="G$1" x="43.18" y="-27.94" smashed="yes" rot="R270">
+<attribute name="NAME" x="48.895" y="-21.59" size="1.778" layer="95" rot="R270"/>
+<attribute name="VALUE" x="38.1" y="-21.59" size="1.778" layer="96" rot="R270"/>
 </instance>
 </instances>
@@
 </segment>
 </net>
-<net name="SP-" class="0">
+<net name="SP+-" class="0">
 <segment>
 <pinref part="U$4" gate="G$1" pin="OUT"/>
@@
 <wire x1="58.42" y1="-5.08" x2="40.64" y2="-5.08" width="0.1524" layer="91"/>
 <junction x="58.42" y="10.16"/>
-<pinref part="JP1" gate="G$1" pin="1"/>
 <wire x1="58.42" y1="-5.08" x2="58.42" y2="-25.4" width="0.1524" layer="91"/>
-<wire x1="58.42" y1="-25.4" x2="38.1" y2="-25.4" width="0.1524" layer="91"/>
 <junction x="58.42" y="-5.08"/>
+<pinref part="JP2" gate="G$1" pin="1"/>
+<wire x1="58.42" y1="-25.4" x2="45.72" y2="-25.4" width="0.1524" layer="91"/>
 </segment>
 </net>
@@
 <pinref part="JP1" gate="G$1" pin="2"/>
 <wire x1="15.24" y1="-5.08" x2="15.24" y2="-25.4" width="0.1524" layer="91"/>
-<wire x1="15.24" y1="-25.4" x2="35.56" y2="-25.4" width="0.1524" layer="91"/>
+<wire x1="15.24" y1="-25.4" x2="25.4" y2="-25.4" width="0.1524" layer="91"/>
 <junction x="15.24" y="-5.08"/>
 </segment>
@@
 </segment>
 </net>
+<net name="SP-" class="0">
+<segment>
+<pinref part="JP2" gate="G$1" pin="2"/>
+<pinref part="JP1" gate="G$1" pin="1"/>
+<wire x1="43.18" y1="-25.4" x2="27.94" y2="-25.4" width="0.1524" layer="91"/>
+<label x="35.56" y="-25.4" size="1.778" layer="95"/>
+</segment>
+</net>

Commit message: Подготовлены платы SP и mtr
Parts:
- added FOTO: VT93N1VERT, KNPN-2023:VT93N1VERT
- added U$7: (no value), KNPN-2023:VIAS-CONNECT
- U$1, U$2: device CanCubeSat:SOLAR-2_1 -> KNPN-2023:SOLAR-2_1
- U$3, U$4: device CanCubeSat:SOLAR-2_0 -> KNPN-2023:SOLAR-2_0
- renumbered JP2 to SP-OUT, LED1 to PWR
Connections:
- net SP+-: now also U$7.1
- net SP-: now also U$7.2
Changed lines of the file:
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@@
 <?xml version="1.0" encoding="utf-8"?>
 <!DOCTYPE eagle SYSTEM "eagle.dtd">
-<eagle version="9.6.2">
+<eagle version="9.4.2">
 <drawing>
 <settings>
-<setting alwaysvectorfont="no"/>
+<setting alwaysvectorfont="yes"/>
 <setting verticaltext="up"/>
 </settings>
@@
 </classes>
 <parts>
-<part name="U$1" library="CanCubeSat" deviceset="SOLAR-2" device="_1" value="SOLAR-2_1"/>
-<part name="U$2" library="CanCubeSat" deviceset="SOLAR-2" device="_1" value="SOLAR-2_1"/>
-<part name="U$3" library="CanCubeSat" deviceset="SOLAR-2" device="_0"/>
-<part name="U$4" library="CanCubeSat" deviceset="SOLAR-2" device="_0"/>
+<part name="U$1" library="KNPN-2023" deviceset="SOLAR-2" device="_1" value="SOLAR-2_1"/>
+<part name="U$2" library="KNPN-2023" deviceset="SOLAR-2" device="_1" value="SOLAR-2_1"/>
+<part name="U$3" library="KNPN-2023" deviceset="SOLAR-2" device="_0"/>
+<part name="U$4" library="KNPN-2023" deviceset="SOLAR-2" device="_0"/>
 <part name="C1" library="rcl" library_urn="urn:adsk.eagle:library:334" deviceset="C-EU" device="C1210" package3d_urn="urn:adsk.eagle:package:23619/2" value="47u"/>
 <part name="R1" library="rcl" library_urn="urn:adsk.eagle:library:334" deviceset="R-US_" device="R0603" package3d_urn="urn:adsk.eagle:package:23555/3" value="2k7"/>
@@
 <part name="D3" library="diode" library_urn="urn:adsk.eagle:library:210" deviceset="MBR0520LT" device="" package3d_urn="urn:adsk.eagle:package:43420/1"/>
 <part name="D4" library="diode" library_urn="urn:adsk.eagle:library:210" deviceset="MBR0520LT" device="" package3d_urn="urn:adsk.eagle:package:43420/1"/>
-<part name="LED1" library="led" library_urn="urn:adsk.eagle:library:259" deviceset="LED" device="CHIP-LED0603" package3d_urn="urn:adsk.eagle:package:15819/3"/>
-<part name="JP2" library="pinhead" library_urn="urn:adsk.eagle:library:325" deviceset="PINHD-1X2" device="" package3d_urn="urn:adsk.eagle:package:22435/2"/>
+<part name="PWR" library="led" library_urn="urn:adsk.eagle:library:259" deviceset="LED" device="CHIP-LED0603" package3d_urn="urn:adsk.eagle:package:15819/3"/>
+<part name="SP-OUT" library="pinhead" library_urn="urn:adsk.eagle:library:325" deviceset="PINHD-1X2" device="" package3d_urn="urn:adsk.eagle:package:22435/2"/>
+<part name="FOTO" library="KNPN-2023" deviceset="VT93N1" device="VERT"/>
+<part name="U$7" library="KNPN-2023" deviceset="VIAS-CONNECT" device=""/>
 </parts>
 <sheets>
@@
 <attribute name="VALUE" x="58.42" y="23.0886" size="1.778" layer="96"/>
 </instance>
-<instance part="LED1" gate="G$1" x="45.72" y="10.16" smashed="yes" rot="R90">
+<instance part="PWR" gate="G$1" x="45.72" y="10.16" smashed="yes" rot="R90">
 <attribute name="NAME" x="50.292" y="13.716" size="1.778" layer="95" rot="R180"/>
 <attribute name="VALUE" x="50.292" y="15.875" size="1.778" layer="96" rot="R180"/>
 </instance>
-<instance part="JP2" gate="G$1" x="43.18" y="-27.94" smashed="yes" rot="R270">
+<instance part="SP-OUT" gate="G$1" x="43.18" y="-27.94" smashed="yes" rot="R270">
 <attribute name="NAME" x="48.895" y="-21.59" size="1.778" layer="95" rot="R270"/>
 <attribute name="VALUE" x="38.1" y="-21.59" size="1.778" layer="96" rot="R270"/>
+</instance>
+<instance part="FOTO" gate="G$1" x="0" y="7.62" smashed="yes" rot="R90">
+<attribute name="NAME" x="0" y="10.16" size="1.778" layer="95" rot="R90"/>
+<attribute name="VALUE" x="2.54" y="10.16" size="1.778" layer="96" rot="R90"/>
+</instance>
+<instance part="U$7" gate="G$1" x="45.72" y="-15.24" smashed="yes" rot="R180">
+<attribute name="NAME" x="49.53" y="-18.415" size="1.778" layer="95" rot="R180"/>
+<attribute name="VALUE" x="49.53" y="-10.795" size="1.778" layer="96" rot="R180"/>
 </instance>
 </instances>
@@
 <wire x1="58.42" y1="33.02" x2="58.42" y2="25.4" width="0.1524" layer="91"/>
 <junction x="58.42" y="33.02"/>
-<pinref part="LED1" gate="G$1" pin="C"/>
+<pinref part="PWR" gate="G$1" pin="C"/>
 <wire x1="58.42" y1="25.4" x2="58.42" y2="10.16" width="0.1524" layer="91"/>
 <wire x1="58.42" y1="10.16" x2="50.8" y2="10.16" width="0.1524" layer="91"/>
@@
 <wire x1="58.42" y1="-5.08" x2="40.64" y2="-5.08" width="0.1524" layer="91"/>
 <junction x="58.42" y="10.16"/>
-<wire x1="58.42" y1="-5.08" x2="58.42" y2="-25.4" width="0.1524" layer="91"/>
+<wire x1="58.42" y1="-5.08" x2="58.42" y2="-15.24" width="0.1524" layer="91"/>
 <junction x="58.42" y="-5.08"/>
-<pinref part="JP2" gate="G$1" pin="1"/>
+<pinref part="SP-OUT" gate="G$1" pin="1"/>
+<wire x1="58.42" y1="-15.24" x2="58.42" y2="-25.4" width="0.1524" layer="91"/>
 <wire x1="58.42" y1="-25.4" x2="45.72" y2="-25.4" width="0.1524" layer="91"/>
+<pinref part="U$7" gate="G$1" pin="1"/>
+<wire x1="48.26" y1="-15.24" x2="58.42" y2="-15.24" width="0.1524" layer="91"/>
+<junction x="58.42" y="-15.24"/>
 </segment>
 </net>
@@
 <segment>
 <pinref part="R1" gate="G$1" pin="2"/>
-<pinref part="LED1" gate="G$1" pin="A"/>
+<pinref part="PWR" gate="G$1" pin="A"/>
 <wire x1="30.48" y1="10.16" x2="43.18" y2="10.16" width="0.1524" layer="91"/>
 </segment>
@@
 <net name="SP-" class="0">
 <segment>
-<pinref part="JP2" gate="G$1" pin="2"/>
+<pinref part="SP-OUT" gate="G$1" pin="2"/>
 <pinref part="JP1" gate="G$1" pin="1"/>
-<wire x1="43.18" y1="-25.4" x2="27.94" y2="-25.4" width="0.1524" layer="91"/>
+<wire x1="43.18" y1="-25.4" x2="35.56" y2="-25.4" width="0.1524" layer="91"/>
 <label x="35.56" y="-25.4" size="1.778" layer="95"/>
-</segment>
-</net>
+<pinref part="U$7" gate="G$1" pin="2"/>
+<wire x1="35.56" y1="-25.4" x2="27.94" y2="-25.4" width="0.1524" layer="91"/>
+<wire x1="43.18" y1="-15.24" x2="35.56" y2="-15.24" width="0.1524" layer="91"/>
+<wire x1="35.56" y1="-15.24" x2="35.56" y2="-25.4" width="0.1524" layer="91"/>
+<junction x="35.56" y="-25.4"/>
+</segment>
+</net>
