File: schematics/board/dop.sch (EAGLE design)
At the start: 42 parts

Commit message: продолжаем делать доп плату
Parts:
- added BUZZER: BUZZERS8R6, CanCubeSat:BUZZERS8R6
- added JP1, JP2: (no value), pinhead:PINHD-2X12
- added JP3, JP4: (no value), pinhead:PINHD-1X3
- added JP5: (no value), pinhead:PINHD-1X2
- added U$10, U$13, U$4: JST_2CON, CanCubeSat:JST_2CON
- added U$12: JST_3CON, CanCubeSat:JST_3CON
- R28, R29: value 10k -> 5k1
- U$1: value BUZZERS8R6 -> JST_2CON; device CanCubeSat:BUZZERS8R6 -> CanCubeSat:JST_2CON
Connections:
- new net CS: JP4.3
- new net CSK: JP4.2
- new net N$23: U$12.2
- new net N$24: U$12.3
- new net N$27: U$10.2
- new net N$28: U$10.1
- new net N$29: U$4.2
- new net N$30: U$4.1
- new net N$31: U$1.2
- new net N$32: U$1.1
- new net N$33: U$13.2
- new net N$34: U$13.1
- new net N$39: JP5.1
- new net N$40: JP5.2
- net 3V3: now also JP3.2
- net 5V: now also BUZZER.VIN, JP3.1; no longer U$1.VIN
- net GND: now also JP3.3
- net MOSI: now also JP4.1
- net N$13: now also BUZZER.GND; no longer U$1.GND
- net PERE1: now also U$12.1

Commit message: добавил фоторезисторы на плату
Parts:
- added R31: 100R, rcl:R-US_0207/15
- added U$11, U$15, U$17, U$18, U$19, U$22, U$23, U$24: VT93N1, CanCubeSat:VT93N1
Connections:
- net N$39 renamed I2C
- net N$40 renamed ADC
- removed net CS: JP4.3
- removed net MOTOR_G: U$21.D
- removed net N$23: U$12.2
- removed net N$24: U$12.3
- removed net N$27: U$10.2
- removed net N$28: U$10.1
- removed net N$29: U$4.2
- removed net N$30: U$4.1
- removed net N$31: U$1.2
- removed net N$32: U$1.1
- removed net N$33: U$13.2
- removed net N$34: U$13.1
- new net MISO: JP2.17
- new net MOTOR3-: U$1.2, U$21.D
- new net PA4: JP2.21
- new net PA5: JP2.24
- new net PA6: JP1.22
- new net PA7: JP1.21
- new net PA8: JP1.4
- new net PC5: JP1.19
- new net SP-: R31.2, U$13.2
- new net VAB: JP1.15, JP2.10
- net 3V3: now also JP1.23, JP2.2
- net 5V: now also JP1.9, JP2.16
- net GND: now also JP1.10, JP1.16, JP1.2, JP1.24, JP2.1, JP2.15, JP2.23, JP2.9
- net INA_SP+: now also R31.1
- net LATCH: now also JP1.12, JP4.3
- net MOSI: now also JP2.18
- net MOTOR1+: now also U$10.1
- net MOTOR1-: now also U$10.2
- net MOTOR2+: now also U$4.1
- net MOTOR2-: now also U$4.2
- net PERE2: now also U$12.2
- net PERE3: now also U$12.3
- net SCK: now also JP2.14
- net SCL: now also JP2.8
- net SDA: now also JP2.7
- net SP+: now also U$13.1
Other:
- moved on the sheet: JP1, JP2

Commit message: я шпион спорадика, почти забацал плату доп
Parts:
- added R30, R32, R33, R34, R35, R36, R37, R38: 2k, rcl:R-US_R0603
- added U$25, U$26, U$27: JST_2CON, CanCubeSat:JST_2CON
- R31: device rcl:R-US_0207/15 -> CanCubeSat:R-US_0207/15
Connections:
- net 3V3: now also R30.2, R32.2, R33.2, R34.2, R35.2, R36.2, R37.2, R38.2
- net FOTO1: now also R32.1, U$17.2
- net FOTO2: now also R34.1, U$11.2
- net FOTO3: now also R30.1, U$18.1
- net FOTO4: now also R35.1, U$19.1
- net FOTO5: now also R36.1, U$22.1
- net FOTO6: now also R38.1, U$24.1
- net FOTO7: now also R37.1, U$23.1
- net FOTO8: now also R33.1, U$15.2
- net GND: now also U$11.1, U$15.1, U$17.1, U$18.2, U$19.2, U$22.2, U$23.2, U$24.2
- net PERE1_G: now also U$25.1
- net PERE2_G: now also U$26.1
- net PERE3_G: now also U$27.1
- net VAB: now also U$25.2, U$26.2, U$27.2
Other:
- moved on the sheet: U$11, U$15, U$17, U$18, U$19, U$22, U$23, U$24

Commit message: Начали делать платы СП
Parts:
- removed U$25, U$26, U$27: JST_2CON, CanCubeSat:JST_2CON
- added ENCODER: JST_3CON, CanCubeSat:JST_3CON
- added FOTO: JST_2CON, CanCubeSat:JST_2CON
- added PERE1, PERE2, PERE3: JST-2-2.5, CanCubeSat:JST-2-2.5
- added X1: 53047-02, con-molex:53047-02
- R12: value 100R -> 1k
- renumbered JP3 to POWER, U$1 to MOT3, U$10 to MOT1, U$12 to PERE-MK, U$13 to SP, U$4 to MOT2
Connections:
- new net ENCOD_A: ENCODER.1
- new net ENCOD_B: ENCODER.2
- new net ENCOD_C: ENCODER.3
- new net FOTO_G: FOTO.2
- new net FOTO_R: FOTO.1
- net GND: now also X1-1.S
- net N$17: now also X1-2.S
- net PERE1_G: now also PERE1.1; no longer U$25.1
- net PERE2_G: now also PERE2.2; no longer U$26.1
- net PERE3_G: now also PERE3.1; no longer U$27.1
- net VAB: now also PERE1.2, PERE2.1, PERE3.2; no longer U$25.2, U$26.2, U$27.2

Commit message: Доделаны платы dop и mtr
Parts:
- removed FOTO, MOT1, MOT2, MOT3: JST_2CON, CanCubeSat:JST_2CON
- removed JP1: (no value), pinhead:PINHD-2X12
- removed JP4, POWER: (no value), pinhead:PINHD-1X3
- removed JP5: (no value), pinhead:PINHD-1X2
- removed PERE-MK: JST_3CON, CanCubeSat:JST_3CON
- removed PERE1, PERE2, PERE3: JST-2-2.5, CanCubeSat:JST-2-2.5
- removed U$21: SI2302CDS, CanCubeSat:SI2302CDS
- removed X1: 53047-02, con-molex:53047-02
- added 74HC595-: 74HC595, CanCubeSat:74HC595
- added A: (no value), pinhead:PINHD-2X12
- added C2, C3: 100nF, rcl:C-USC0603
- added LED, LED1: MOLEX-3-1.25, CanCubeSat:MOLEX-3-1.25
- added MOT-H, MOT-ST, MOT-V, PHOTO: MOLEX-2-1.25, CanCubeSat:MOLEX-2-1.25
- added PER-PAR, PER-SP, PER-ST: JST-2-2.5, CanCubeSat:JST-2-2.5
- added R39: 2k, rcl:R-US_R0603
- added R41: 100R, rcl:R-US_R0603
- added R42: 4k7, rcl:R-US_R0603
- added SI2302: SI2302CDS, CanCubeSat:SI2302CDS
- ENCODER: value JST_3CON -> MOLEX-3-1.25; device CanCubeSat:JST_3CON -> CanCubeSat:MOLEX-3-1.25
- R11: value 10k -> 5k1
- R12: value 1k -> 5k1
- R16: value 10k -> 10k*3
- SP: value JST_2CON -> MOLEX-2-1.25; device CanCubeSat:JST_2CON -> CanCubeSat:MOLEX-2-1.25
- U$11, U$15, U$17, U$18, U$19, U$22, U$23, U$24: device CanCubeSat:VT93N1 -> KNPN-2023:VT93N1
- renumbered JP2 to B, U$14 to IRF7905, U$16 to AD5593, U$2 to INA, U$20 to SI2302-, U$3 to 74HC595, U$5 to IRF7905-, U$6 to AP9930, U$7 to NDC7002, U$8 to AP9930-, U$9 to NDC7002-
Connections:
- removed net ADC: JP5.2
- removed net CSK: JP4.2
- removed net ENCOD_C: ENCODER.3
- removed net FOTO_G: FOTO.2
- removed net FOTO_R: FOTO.1
- removed net I2C: JP5.1
- removed net MOTOR3-: MOT3.2, U$21.D
- removed net N$10: IRF7905.S2, R21.2
- removed net N$11: IRF7905.G1, R20.2, R23.1
- removed net N$19: IRF7905-.S2, R25.2
- removed net PA4: B.21
- removed net PA5: B.24
- removed net PA7: JP1.21
- removed net PA8: JP1.4
- new net FOTO9: A.22, PHOTO.1, R39.1
- new net LED: A.3, R41.1
- new net N$22: 74HC595-.DS, 74HC595.Q7S
- new net N$23: LED.2, LED1.2, R42.2, SI2302.D
- net 3V3: now also 74HC595-.MR, 74HC595-.VCC, A.24, B.1, R11.2, R12.2, R39.2; no longer B.2, JP1.23, POWER.2
- net 5V: now also A.10, B.15, LED.1, LED1.1, R42.1; no longer B.16, JP1.9, POWER.1
- net BUZZER: now also 74HC595-.Q1
- net ENCOD_A: now also B.22, C3.2, R11.1
- net ENCOD_B: now also B.23, C2.2, ENCODER.3, R12.1; no longer ENCODER.2
- net FOTO2: now also U$11.1; no longer U$11.2
- net FOTO3: now also U$18.2; no longer U$18.1
- net FOTO6: now also U$24.2; no longer U$24.1
- net GND: now also 74HC595-.GND, 74HC595-.OE, A.1, A.15, A.23, A.9, B.10, B.16, B.2, B.24, C2.1, C3.1, ENCODER.2, IRF7905-.S2, IRF7905.G1, IRF7905.S2, LED.3, LED1.3, MOT-ST.2, PHOTO.2, R20.2, R21.2, R23.1, R25.2, SI2302.S, U$11.2, U$18.1, U$24.1; no longer B.1, B.15, B.23, B.9, JP1.10, JP1.16, JP1.2, JP1.24, POWER.3, R11.2, U$11.1, U$18.2, U$21.S, U$24.2, X1-1.S
- net LATCH: now also 74HC595-.STCP, A.11; no longer JP1.12, JP4.3
- net MISO: now also B.18; no longer B.17
- net MOSI: now also B.17; no longer B.18, JP4.1
- net MOTOR1+: now also MOT-H.2; no longer MOT1.1
- net MOTOR1-: now also MOT-H.1; no longer MOT1.2
- net MOTOR2+: now also MOT-V.2; no longer MOT2.1
- net MOTOR2-: now also MOT-V.1; no longer MOT2.2
- net N$17: now also R41.2, SI2302.G; no longer R11.1, R12.2, U$21.G, X1-2.S
- net PA6: now also A.21; no longer JP1.22
- net PC5: now also A.20; no longer JP1.19
- net PERE1: no longer PERE-MK.1
- net PERE1_G: now also PER-PAR.1; no longer PERE1.1
- net PERE2: no longer PERE-MK.2
- net PERE2_G: now also PER-ST.1; no longer PERE2.2
- net PERE3: no longer PERE-MK.3
- net PERE3_G: now also PER-SP.1; no longer PERE3.1
- net SCK: now also 74HC595-.SHCP, B.13; no longer B.14
- net SCL: now also B.7; no longer B.8
- net SDA: now also B.8; no longer B.7
- net TRUBKI: now also MOT-ST.1; no longer R12.1
- net VAB: now also A.16, B.9, PER-PAR.2, PER-SP.2, PER-ST.2; no longer B.10, JP1.15, PERE1.2, PERE2.1, PERE3.2
Other:
- moved on the sheet: R11, R12, R36, R37, R38, U$11, U$18, U$22, U$23, U$24

Commit message: Подготовлена плата dop
Parts:
- added R40: 10k, rcl:R-US_R0603
Connections:
- removed net PA6: A.21
- removed net PC5: A.20
- new net SWITCH: B.22, R40.1
- net 3V3: now also R40.2
- net ENCOD_A: now also A.21; no longer B.22
- net ENCOD_B: now also A.22; no longer B.23
- net FOTO9: now also B.23; no longer A.22
Changed lines of the file:
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@@
 <part name="R42" library="rcl" library_urn="urn:adsk.eagle:library:334" deviceset="R-US_" device="R0603" package3d_urn="urn:adsk.eagle:package:23555/3" value="4k7"/>
 <part name="74HC595-" library="CanCubeSat" deviceset="74HC595" device=""/>
+<part name="R40" library="rcl" library_urn="urn:adsk.eagle:library:334" deviceset="R-US_" device="R0603" package3d_urn="urn:adsk.eagle:package:23555/3" value="10k"/>
 </parts>
 <sheets>
@@
 </instance>
 <instance part="74HC595-" gate="G$1" x="322.58" y="-76.2" smashed="yes"/>
+<instance part="R40" gate="G$1" x="91.44" y="-254" smashed="yes" rot="R180">
+<attribute name="NAME" x="95.25" y="-255.4986" size="1.778" layer="95" rot="R180"/>
+<attribute name="VALUE" x="95.25" y="-250.698" size="1.778" layer="96" rot="R180"/>
+</instance>
 </instances>
 <busses>
@@
 </segment>
 <segment>
-<wire x1="-58.42" y1="-187.96" x2="-45.72" y2="-187.96" width="0.1524" layer="91"/>
-<label x="-58.42" y="-187.96" size="1.778" layer="95"/>
+<wire x1="-60.96" y1="-187.96" x2="-45.72" y2="-187.96" width="0.1524" layer="91"/>
+<label x="-60.96" y="-187.96" size="1.778" layer="95"/>
 <pinref part="A" gate="A" pin="10"/>
 </segment>
@@
 </segment>
 <segment>
-<wire x1="-58.42" y1="-205.74" x2="-45.72" y2="-205.74" width="0.1524" layer="91"/>
-<label x="-58.42" y="-205.74" size="1.778" layer="95"/>
+<wire x1="-60.96" y1="-205.74" x2="-45.72" y2="-205.74" width="0.1524" layer="91"/>
+<label x="-60.96" y="-205.74" size="1.778" layer="95"/>
 <pinref part="A" gate="A" pin="24"/>
 </segment>
@@
 <label x="337.82" y="-68.58" size="1.778" layer="95"/>
 <pinref part="74HC595-" gate="G$1" pin="VCC"/>
+</segment>
+<segment>
+<pinref part="R40" gate="G$1" pin="2"/>
+<wire x1="86.36" y1="-254" x2="76.2" y2="-254" width="0.1524" layer="91"/>
+<label x="76.2" y="-254" size="1.778" layer="95"/>
 </segment>
 </net>
@@
 </segment>
 <segment>
-<wire x1="-58.42" y1="-195.58" x2="-45.72" y2="-195.58" width="0.1524" layer="91"/>
-<label x="-58.42" y="-195.58" size="1.778" layer="95"/>
+<wire x1="-60.96" y1="-195.58" x2="-45.72" y2="-195.58" width="0.1524" layer="91"/>
+<label x="-60.96" y="-195.58" size="1.778" layer="95"/>
 <pinref part="A" gate="A" pin="16"/>
 </segment>
@@
 </segment>
 <segment>
-<wire x1="-12.7" y1="-203.2" x2="2.54" y2="-203.2" width="0.1524" layer="91"/>
-<label x="-12.7" y="-203.2" size="1.778" layer="95"/>
-<pinref part="B" gate="A" pin="22"/>
+<wire x1="-22.86" y1="-203.2" x2="-38.1" y2="-203.2" width="0.1524" layer="91"/>
+<label x="-30.48" y="-203.2" size="1.778" layer="95"/>
+<pinref part="A" gate="A" pin="21"/>
 </segment>
 </net>
@@
 </segment>
 <segment>
-<wire x1="22.86" y1="-205.74" x2="10.16" y2="-205.74" width="0.1524" layer="91"/>
-<label x="17.78" y="-205.74" size="1.778" layer="95"/>
-<pinref part="B" gate="A" pin="23"/>
+<wire x1="-60.96" y1="-203.2" x2="-45.72" y2="-203.2" width="0.1524" layer="91"/>
+<label x="-60.96" y="-203.2" size="1.778" layer="95"/>
+<pinref part="A" gate="A" pin="22"/>
 </segment>
 </net>
@@
 </segment>
 <segment>
-<wire x1="-58.42" y1="-203.2" x2="-45.72" y2="-203.2" width="0.1524" layer="91"/>
-<label x="-58.42" y="-203.2" size="1.778" layer="95"/>
-<pinref part="A" gate="A" pin="22"/>
-</segment>
-</net>
-<net name="PA6" class="0">
-<segment>
-<wire x1="-22.86" y1="-203.2" x2="-38.1" y2="-203.2" width="0.1524" layer="91"/>
-<label x="-30.48" y="-203.2" size="1.778" layer="95"/>
-<pinref part="A" gate="A" pin="21"/>
-</segment>
-</net>
-<net name="PC5" class="0">
-<segment>
-<wire x1="-58.42" y1="-200.66" x2="-45.72" y2="-200.66" width="0.1524" layer="91"/>
-<label x="-58.42" y="-200.66" size="1.778" layer="95"/>
-<pinref part="A" gate="A" pin="20"/>
+<wire x1="22.86" y1="-205.74" x2="10.16" y2="-205.74" width="0.1524" layer="91"/>
+<label x="17.78" y="-205.74" size="1.778" layer="95"/>
+<pinref part="B" gate="A" pin="23"/>
 </segment>
 </net>
@@
 </segment>
 </net>
+<net name="SWITCH" class="0">
+<segment>
+<wire x1="-12.7" y1="-203.2" x2="2.54" y2="-203.2" width="0.1524" layer="91"/>
+<label x="-12.7" y="-203.2" size="1.778" layer="95"/>
+<pinref part="B" gate="A" pin="22"/>
+</segment>
+<segment>
+<pinref part="R40" gate="G$1" pin="1"/>
+<wire x1="96.52" y1="-254" x2="109.22" y2="-254" width="0.1524" layer="91"/>
+<label x="101.6" y="-254" size="1.778" layer="95"/>
+</segment>
+</net>
