File: schematics/board/zakaz 2/dop.brd (EAGLE design)
At the start: 65.8 x 65.8 mm, 79 parts

Commit message: Новые версии плат
Parts:
- removed AP9930, AP9930-: AP9930GM, CanCubeSat:SO8
- removed NDC7002, NDC7002-: NDC7002N, CanCubeSat:SOT23-6
- added R43: 10k, rcl:R0603
- added SI2302-1, SI2302-2, SI2302-3, SI2302-4: SI2302CDS, CanCubeSat:SOT23-3
- added U$1, U$2, U$3, U$4: FDC6420C, KNPN-2023:TSOP-6
- R16: value 10k*3 -> 10k
- moved R8 14.4 mm to (18.0, 42.7)
- moved R3 14.1 mm to (18.1, 51.0)
- moved R16 10.6 mm to (28.7, 53.4)
- moved R7 8.80 mm to (20.5, 45.3), turned to 180 degrees
- moved R6 7.94 mm to (20.9, 40.3)
- moved R1 7.93 mm to (20.6, 53.3), turned to 180 degrees
- moved R17 7.26 mm to (20.9, 48.3)
- moved R5 6.75 mm to (28.7, 45.2), turned to 0 degrees
- moved R4 1.94 mm to (31.5, 51.0)
- moved R12 1.56 mm to (29.0, 57.8), turned to 180 degrees
- moved R18 1.30 mm to (31.4, 42.6)
- moved R11 1.20 mm to (25.9, 57.8), turned to 0 degrees
- moved C2 1.02 mm to (29.0, 59.9), turned to 0 degrees
- moved B 1.00 mm to (53.2, 33.0)
- moved R19 0.71 mm to (28.8, 40.2)
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Connections:
- removed net N$2: AP9930.1, AP9930.8, NDC7002.6, R16.1, R2.1
- removed net N$4: AP9930.4, AP9930.5, NDC7002.4, R1.1, R17.1
- removed net N$9: IRF7905.3, R20.1
- new net N$10: IRF7905.4, R20.2, R23.1
- new net N$19: R17.1, SI2302-3.3, U$2.P$1, U$2.P$3
- new net N$24: R16.1, SI2302-1.3, U$1.P$1, U$1.P$3
- net 5V: now also U$1.P$2, U$2.P$2, U$3.P$2, U$4.P$2; no longer AP9930-.7, AP9930.7
- net GND: now also IRF7905.3, R1.1, R19.1, R2.1, R20.1, R43.1, R7.1, SI2302-1.2, SI2302-2.2, SI2302-3.2, SI2302-4.2, U$1.P$5, U$2.P$5, U$3.P$5, U$4.P$5; no longer AP9930-.3, AP9930.3, IRF7905.4, NDC7002-.2, NDC7002-.5, NDC7002.2, NDC7002.5, R20.2, R23.1
- net MOTOR1+: now also U$4.P$4, U$4.P$6; no longer AP9930-.6
- net MOTOR1-: now also U$3.P$4, U$3.P$6; no longer AP9930-.2
- net MOTOR2+: now also U$2.P$4, U$2.P$6; no longer AP9930.6
- net MOTOR2-: now also U$1.P$4, U$1.P$6; no longer AP9930.2
- net N$1: now also SI2302-3.1; no longer NDC7002.3
- net N$17: now also R43.2
- net N$3: now also SI2302-1.1; no longer NDC7002.1
- net N$5: now also SI2302-2.3, U$3.P$1, U$3.P$3; no longer AP9930-.1, AP9930-.8, NDC7002-.6, R19.1
- net N$6: now also SI2302-4.1; no longer NDC7002-.3
- net N$7: now also SI2302-2.1; no longer NDC7002-.1
- net N$8: now also SI2302-4.3, U$4.P$1, U$4.P$3; no longer AP9930-.4, AP9930-.5, NDC7002-.4, R7.1
Routing:
- net GND: track 507.3 -> 551.8 mm, vias 11 -> 10
- net MK_MOTOR1+: track 9.03 -> 41.0 mm, vias 0 -> 2
- net MK_MOTOR2+: track 3.53 -> 24.1 mm
- net 5V: track 126.8 -> 143.8 mm, vias 7 -> 5
- net N$2: track 12.2 -> 0.00 mm
- net N$4: track 11.6 -> 0.00 mm
- net N$24: track 0.00 -> 7.87 mm
- net N$19: track 0.00 -> 7.80 mm
- net N$5: track 12.5 -> 7.80 mm
- net N$10: track 0.00 -> 4.40 mm
- net N$8: track 11.7 -> 7.80 mm
- net 3V3: track 240.7 -> 242.8 mm
- net N$9: track 2.12 -> 0.00 mm
- net N$1: track 4.87 -> 3.32 mm
- net N$17: track 1.90 -> 3.30 mm
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Other:
- board text added: "100nF*2"
- board text added: "5k1*2"
- board text added: "FDC*4"
- board text added: "SI*2"
