File: schematics/board/zakaz 2/dop.sch (EAGLE design)
At the start: 79 parts

Commit message: Новые версии плат
Parts:
- removed AP9930, AP9930-: AP9930GM, CanCubeSat:AP9930GM
- removed NDC7002, NDC7002-: NDC7002N, CanCubeSat:NDC7002N
- added R43: 10k, rcl:R-US_R0603
- added SI2302-1, SI2302-2, SI2302-3, SI2302-4: SI2302CDS, CanCubeSat:SI2302CDS
- added U$1, U$2, U$3, U$4: FDC6420C, KNPN-2023:FDC6420C
- R16: value 10k*3 -> 10k
Connections:
- removed net N$2: AP9930.N1G, AP9930.P1G, NDC7002.D1, R16.1, R2.1
- removed net N$4: AP9930.N2G, AP9930.P2G, NDC7002.D2, R1.1, R17.1
- removed net N$9: IRF7905.S1, R20.1
- new net N$10: IRF7905.G1, R20.2, R23.1
- new net N$19: R17.1, SI2302-3.D, U$2.NG, U$2.PG
- new net N$24: R16.1, SI2302-1.D, U$1.NG, U$1.PG
- net 5V: now also U$1.PS, U$2.PS, U$3.PS, U$4.PS; no longer AP9930-.PS, AP9930.PS
- net GND: now also IRF7905.S1, R1.1, R19.1, R2.1, R20.1, R43.1, R7.1, SI2302-1.S, SI2302-2.S, SI2302-3.S, SI2302-4.S, U$1.NS, U$2.NS, U$3.NS, U$4.NS; no longer AP9930-.NS, AP9930.NS, IRF7905.G1, NDC7002-.S1, NDC7002-.S2, NDC7002.S1, NDC7002.S2, R20.2, R23.1
- net MOTOR1+: now also U$4.ND, U$4.PD; no longer AP9930-.P2N2D
- net MOTOR1-: now also U$3.ND, U$3.PD; no longer AP9930-.P1N1D
- net MOTOR2+: now also U$2.ND, U$2.PD; no longer AP9930.P2N2D
- net MOTOR2-: now also U$1.ND, U$1.PD; no longer AP9930.P1N1D
- net N$1: now also SI2302-3.G; no longer NDC7002.G2
- net N$17: now also R43.2
- net N$3: now also SI2302-1.G; no longer NDC7002.G1
- net N$5: now also SI2302-2.D, U$3.NG, U$3.PG; no longer AP9930-.N1G, AP9930-.P1G, NDC7002-.D1, R19.1
- net N$6: now also SI2302-4.G; no longer NDC7002-.G2
- net N$7: now also SI2302-2.G; no longer NDC7002-.G1
- net N$8: now also SI2302-4.D, U$4.NG, U$4.PG; no longer AP9930-.N2G, AP9930-.P2G, NDC7002-.D2, R7.1
Other:
- moved on the sheet: R1, R16, R17, R18, R19, R2, R3, R4, R5, R6, R7, R8
